Commit message: added prefix let's fix that later

File: pf3400_description/urdf/macro.gazebo.xacro (robot description, xacro)
@@ -1,5 +1,5 @@
 <?xml version="1.0"?>
 <robot xmlns:xacro="http://www.ros.org/wiki/xacro">
-  <xacro:macro name="pf3400_gazebo" params="ns">
+  <xacro:macro name="pf3400_gazebo" params="ns prefix">
     <gazebo reference="z_column">
       <selfCollide>true</selfCollide>
