Commit message: fixed file for the demo purposes

File: pf3400_description/urdf/PF3400SX.urdf (robot description, URDF)
Before this commit: robot PF3400SX Robot, 7 links, 6 joints
Links:
- link hand: geometry visual mesh filename=package://pf3400_description/meshes/PF3400_Hand.STL scale=0.001 0.001 0.001
- link inner_link: geometry visual mesh filename=package://pf3400_description/meshes/PF3400_Inner_Link.STL scale=0.001 0.001 0.001
- link left_finger: geometry visual mesh filename=package://pf3400_description/meshes/PF3400_Left_Finger.STL scale=0.001 0.001 0.001
- link outer_link: geometry visual mesh filename=package://pf3400_description/meshes/PF3400_Outer_Link.STL scale=0.001 0.001 0.001
- link right_finger: geometry visual mesh filename=package://pf3400_description/meshes/PF3400_Right_Finger.STL scale=0.001 0.001 0.001
- link z_carriage: geometry visual mesh filename=package://pf3400_description/meshes/PF3400_Z_Carriage.STL scale=0.001 0.001 0.001
- link z_column: geometry visual mesh filename=package://pf3400_description/meshes/PF3400_Z_Column.STL scale=0.001 0.001 0.001
